Commit message: add xbot

File: resources/robots/hi/urdf/hi_1_21_240815_rl.urdf (robot description, URDF)
Before this commit: robot hi_1_21_240815, 22 links, 21 joints
Links:
- link base_link: mass 0.67789918 -> 3.67

File: resources/robots/x1_14DOF/meshes/x1_14DOF.urdf (robot description, URDF)
Before this commit: robot x1, 58 links, 57 joints
Links:
- link base_link: geometry collision mesh filename=../meshes/base_link_simple.STL; visual mesh filename=../meshes/base_link_simple.STL
Joints:
- joint left_elbow_pitch_joint: limit lower=-3.14 upper=3.14 effort=0 velocity=0 -> lower=-1.7 upper=1.7 effort=0 velocity=0
- joint left_hip_pitch_joint: origin xyz=0.00110 0.092277 -0.023143 rpy=0 -1.5708 1.5708 -> xyz=0.00245 0.092277 -0.012143 rpy=0 -0.7854 1.5708
- joint left_hip_roll_joint: origin xyz=0 -0.0405000000000076 -0.0589000000000007 rpy=1.57079632679491 1.57079632679491 0 -> xyz=0 -0.0405000000000076 -0.0589000000000007 rpy=1.57079632679491 0.785398163397451 0
- joint left_shoulder_pitch_joint: limit lower=-3.14 upper=3.14 effort=0 velocity=0 -> lower=-3.14 upper=3.14 effort=30 velocity=10; type fixed -> revolute
- joint right_elbow_pitch_joint: limit lower=-3.14 upper=3.14 effort=0 velocity=0 -> lower=-1.7 upper=1.7 effort=0 velocity=0
- joint right_hip_pitch_joint: origin xyz=0.00110 -0.092277 -0.023143 rpy=0 -1.5708 -1.5708 -> xyz=0.00245 -0.092277 -0.012143 rpy=0 -0.7854 -1.5708
- joint right_hip_roll_joint: origin xyz=0 0.0405000000001067 -0.0588999999999981 rpy=1.57079632679491 1.57079632679491 0 -> xyz=0 0.0405000000001067 -0.0588999999999981 rpy=1.57079632679491 0.78539816339745 0
- joint right_shoulder_pitch_joint: limit lower=-3.14 upper=3.14 effort=0 velocity=0 -> lower=-3.14 upper=3.14 effort=30 velocity=10; type fixed -> revolute
- joint right_shoulder_roll_joint: limit lower=-3.14 upper=3.14 effort=0 velocity=0 -> lower=-3.14 upper=3.14 effort=30 velocity=10
